File: SolarCell+Y.sch (KiCad schematic (older format))
At the start: 28 parts, among them IC1 symbols_TSL2561, J1 symbols_XF2M-1015-1A, J2 U.FL-R-SMT-1, Q1 IRLML2803, U1 HHM17139B2, U2 NDS8434

Commit message: UFL added. Another footprint victory.
Parts:
- J2: footprint U.FL-R-SMT-1 -> Connector_Coaxial:U.FL_Hirose_U.FL-R-SMT-1_Vertical
Changed lines of the file:
@@
 F 0 "J2" H 2178 6738 50  0000 L CNN
 F 1 "U.FL-R-SMT-1" H 2178 6647 50  0000 L CNN
-F 2 "U.FL-R-SMT-1" H 1650 7050 50  0001 L CNN
+F 2 "Connector_Coaxial:U.FL_Hirose_U.FL-R-SMT-1_Vertical" H 1650 7050 50  0001 L CNN
 F 3 "https://www.hirose.co.jp/cataloge_hp/ed_UFL_20141014.pdf" H 1650 6950 50  0001 L CNN
 F 4 "Hirose" H 1650 6650 50  0001 L CNN "Manufacturer_Name"

Commit message: Caught mistake on burnwire circuit.
Parts:
- R5: value 10k -> 1M
- R7: value 100k -> 1M
Connections:
- wire segments 70 -> 75
Other:
- moved on the sheet: R5
Changed lines of the file:
@@
 Text Notes 7700 4600 0    157  ~ 0
 Burnwire Control\n\n
-Wire Wire Line
-	8100 5600 8400 5600
 Text Label 10550 5300 2    50   ~ 0
 VBURN
@@
 Text GLabel 8000 5200 0    50   BiDi ~ 0
 BURN1
-Connection ~ 8100 5200
 Wire Wire Line
-	8800 5500 8800 5600
-Wire Wire Line
-	8500 5400 8500 5200
+	8500 5400 8500 5300
 Wire Wire Line
 	8800 5100 9150 5100
@@
 AR Path="/5CEC6476/5DB28BB7" Ref="R?"  Part="1"
 F 0 "R7" V 8861 5232 70  0000 R CNN
-F 1 "100k" V 8740 5232 70  0000 R CNN
+F 1 "1M" V 8740 5232 70  0000 R CNN
 F 2 "Resistor_SMD:R_0402_1005Metric" H 8800 5300 50  0001 C CNN
 F 3 "" H 8800 5300 50  0001 C CNN
 	1    8800 5300
 	0    -1   -1   0
-$EndComp
-$Comp
-L SolarCell+Y-rescue:RESISTOR0603-mainboard-misc-circuits-rescue-SolarCellZ_v1-rescue R5
-U 1 1 5DB28BC9
-P 8100 5400
-AR Path="/5DB28BC9" Ref="R5"  Part="1"
-AR Path="/5CEC6476/5DB28BC9" Ref="R?"  Part="1"
-F 0 "R5" V 8039 5333 70  0000 R CNN
-F 1 "10k" V 8160 5333 70  0000 R CNN
-F 2 "Resistor_SMD:R_0402_1005Metric" H 8100 5400 50  0001 C CNN
-F 3 "" H 8100 5400 50  0001 C CNN
-	1    8100 5400
-	0    1    1    0
 $EndComp
 $Comp
@@
 	1    8300 5200
 	-1   0    0    1
-$EndComp
-$Comp
-L SolarCell+Y-rescue:IRLML2803TRPBF-mainboard-misc-circuits-rescue-SolarCellZ_v1-rescue Q1
-U 1 1 5DB28BE3
-P 8600 5500
-AR Path="/5DB28BE3" Ref="Q1"  Part="1"
-AR Path="/5CEC6476/5DB28BE3" Ref="Q?"  Part="1"
-F 0 "Q1" V 8850 5500 59  0000 C CNN
-F 1 "IRLML2803" V 8950 5600 59  0000 C CNN
-F 2 "Package_TO_SOT_SMD:SOT-23" H 8600 5500 50  0001 C CNN
-F 3 "" H 8600 5500 50  0001 C CNN
-F 4 "2302" V 8600 5500 50  0001 C CNN "Proto"
-F 5 "IRLML2803" V 8600 5500 50  0001 C CNN "Flight"
-	1    8600 5500
-	0    1    1    0
 $EndComp
 $Comp
@@
 Wire Wire Line
 	9150 5700 8800 5700
-Wire Wire Line
-	8800 5700 8800 5600
-Connection ~ 8800 5600
 Wire Wire Line
 	9150 5500 9150 5300
@@
 	1    0    0    -1
 $EndComp
-$Comp
-L power:GND #PWR0108
-U 1 1 5DB4839B
-P 8100 5600
-F 0 "#PWR0108" H 8100 5350 50  0001 C CNN
-F 1 "GND" H 8105 5427 50  0000 C CNN
-F 2 "" H 8100 5600 50  0001 C CNN
-F 3 "" H 8100 5600 50  0001 C CNN
-	1    8100 5600
-	1    0    0    -1
-$EndComp
-Connection ~ 8100 5600
 Wire Wire Line
 	8800 5100 7250 5100
@@
 Text GLabel 7250 5100 0    50   BiDi ~ 0
 BATT_P
+$Comp
+L power:GND #PWR0108
+U 1 1 5DB4839B
+P 8200 5750
+F 0 "#PWR0108" H 8200 5500 50  0001 C CNN
+F 1 "GND" H 8205 5577 50  0000 C CNN
+F 2 "" H 8200 5750 50  0001 C CNN
+F 3 "" H 8200 5750 50  0001 C CNN
+	1    8200 5750
+	1    0    0    -1
+$EndComp
+$Comp
+L SolarCell+Y-rescue:RESISTOR0603-mainboard-misc-circuits-rescue-SolarCellZ_v1-rescue R5
+U 1 1 5DB28BC9
+P 8200 5500
+AR Path="/5DB28BC9" Ref="R5"  Part="1"
+AR Path="/5CEC6476/5DB28BC9" Ref="R?"  Part="1"
+F 0 "R5" V 8139 5433 70  0000 R CNN
+F 1 "1M" V 8260 5433 70  0000 R CNN
+F 2 "Resistor_SMD:R_0402_1005Metric" H 8200 5500 50  0001 C CNN
+F 3 "" H 8200 5500 50  0001 C CNN
+	1    8200 5500
+	0    1    1    0
+$EndComp
+Connection ~ 8800 5600
+Wire Wire Line
+	8800 5700 8800 5600
+Wire Wire Line
+	8800 5500 8800 5600
+$Comp
+L SolarCell+Y-rescue:IRLML2803TRPBF-mainboard-misc-circuits-rescue-SolarCellZ_v1-rescue Q1
+U 1 1 5DB28BE3
+P 8600 5500
+AR Path="/5DB28BE3" Ref="Q1"  Part="1"
+AR Path="/5CEC6476/5DB28BE3" Ref="Q?"  Part="1"
+F 0 "Q1" V 8850 5500 59  0000 C CNN
+F 1 "IRLML2803" V 8950 5600 59  0000 C CNN
+F 2 "Package_TO_SOT_SMD:SOT-23" H 8600 5500 50  0001 C CNN
+F 3 "" H 8600 5500 50  0001 C CNN
+F 4 "2302" V 8600 5500 50  0001 C CNN "Proto"
+F 5 "IRLML2803" V 8600 5500 50  0001 C CNN "Flight"
+	1    8600 5500
+	0    1    1    0
+$EndComp
+Wire Wire Line
+	8200 5300 8500 5300
+Connection ~ 8500 5300
+Wire Wire Line
+	8500 5300 8500 5200
+Wire Wire Line
+	8400 5600 8300 5600
+Wire Wire Line
+	8300 5600 8300 5700
+Wire Wire Line
+	8300 5700 8200 5700
+Wire Wire Line
+	8200 5700 8200 5750
+Connection ~ 8200 5700
 $EndSCHEMATC

Commit message: v01 order + repo update
Parts:
- removed IC1: symbols_TSL2561, TSL2561, symbol SolarCell+Y-rescue:symbols_TSL2561-misc-circuits-cache
- removed J2: U.FL-R-SMT-1, Connector_Coaxial:U.FL_Hirose_U.FL-R-SMT-1_Vertical, symbol SolarCell+Y-rescue:U.FL-R-SMT-1-symbols
- removed U1: HHM17139B2, custom-footprints:balun0603, symbol SolarCell+Y-rescue:HHM17139B2-symbols
- added J2: U.FL-R-SMT-1, custom-footprints:U.FL-R-SMT-1, symbol symbols:U.FL-R-SMT-1
- added R10, R8, R9: 0, Resistor_SMD:R_0402_1005Metric, symbol Device:R_Small_US
- added TP1, TP2, TP3, TP4, TP5: TP, TestPoint:TestPoint_THTPad_D1.0mm_Drill0.5mm, symbol Connector:TestPoint
- added U1: TTB12G51-Balun, custom-footprints:TTB12G51-balun, symbol symbols:TTB12G51-Balun
- added U3: TSL2561, custom-footprints:TSL2561, symbol symbols:TSL2561
- C1: footprint (none) -> Capacitor_SMD:C_0402_1005Metric
- JP1: footprint SolarCellParts:Burn-Wire-Rotated -> custom-footprints:Burn-Wire
- SC1, SC2, SC3, SC4, SC5, SC6, SC7, SC8: footprint SolarCellParts:KXOB25-05X3F -> custom-footprints:KXOB25-05X3F
Connections:
- wire segments 75 -> 77
Other:
- note added: "COIL+\n"
- note added: "COIL-\n"
- note added: "Clockwise\n(while facing layer 1)"
- moved on the sheet: H1, H2, J1

Commit message: repaired schematic such that it matches pcb. repaired pcb such that design rules are met
Parts:
- removed R4: 0, Resistor_SMD:R_0402_1005Metric, symbol Device:R_Small_US
- added C10, C15, C9: 0.1uF, Capacitor_SMD:C_0402_1005Metric, symbol SolarCellX_v3-rescue:0.1UF-0603-25V-(+80_-20%)-misc-circuits-cache-misc-circuit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
- added C11, C12, C14, C6: 100uF, Capacitor_SMD:C_0603_1608Metric, symbol SolarCellX_v3-rescue:0.1UF-0603-25V-(+80_-20%)-misc-circuits-cache-misc-circuit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
- added C2: 1.0uF, Capacitor_SMD:C_0402_1005Metric, symbol SolarCellX_v3-rescue:1.0UF-0603-16V-10%-misc-circuits-cache-misc-circuits-rescue
- added C3, C8: 4.7uF, Capacitor_SMD:C_0402_1005Metric, symbol SolarCellX_v3-rescue:4.7UF0603-misc-circuits-cache-misc-circuits-rescue
- added C4: 10nF, Capacitor_SMD:C_0402_1005Metric, symbol SolarCellX_v3-rescue:10NF-0603-50V-10%-misc-circuits-cache-misc-circuits-rescue
- added C7: 22uF, Capacitor_SMD:C_0402_1005Metric, symbol SolarCellX_v3-rescue:22UF-0805-6.3V-20%-misc-circuits-cache-misc-circuits-rescue
- added D4: MSS1P4-M3_89A, misc-circuits:MICROSMP, symbol SolarCellX_v3-rescue:MSS1P4-M3_89A-symbols
- added D5: SDM20U40-7, misc-circuits:SOD523, symbol SolarCellX_v3-rescue:DIODE-SOD523-misc-circuits-cache-misc-circuits-rescue
- added L1: 22uH-LPS4018-223MR, misc-circuits:LPS4018, symbol SolarCellX_v3-rescue:COILCRAFT-LPS4018-misc-circuits-cache-misc-circuits-rescue
- added L2: 10uH-LPS4018-103MR, misc-circuits:LPS4018, symbol SolarCellX_v3-rescue:COILCRAFT-LPS4018-misc-circuits-cache-misc-circuits-rescue
- added R11: 4.75M, Resistor_SMD:R_0402_1005Metric, symbol SolarCellX_v3-rescue:1MOHM-0603-1_4W-5%-misc-circuits-cache-misc-circuits-rescue
- added R12, R18: 8.25M, Resistor_SMD:R_0402_1005Metric, symbol SolarCellX_v3-rescue:1MOHM-0603-1_4W-5%-misc-circuits-cache-misc-circuits-rescue
- added R13, R14, R20, R21, R25, R4: 0, Resistor_SMD:R_0402_1005Metric, symbol SolarCellX_v3-rescue:0OHM-0603-1_10W-5%-misc-circuits-cache-misc-circuits-rescue
- added R15: 7.32M, Resistor_SMD:R_0402_1005Metric, symbol SolarCellX_v3-rescue:1MOHM-0603-1_4W-5%-misc-circuits-cache-misc-circuits-rescue
- added R16: 5.62M, Resistor_SMD:R_0402_1005Metric, symbol SolarCellX_v3-rescue:1MOHM-0603-1_4W-5%-misc-circuits-cache-misc-circuits-rescue
- added R17: 374K, Resistor_SMD:R_0402_1005Metric, symbol SolarCellX_v3-rescue:1MOHM-0603-1_4W-5%-misc-circuits-cache-misc-circuits-rescue
- added R19: 4.53M, Resistor_SMD:R_0402_1005Metric, symbol SolarCellX_v3-rescue:1MOHM-0603-1_4W-5%-misc-circuits-cache-misc-circuits-rescue
- added U4: Value, misc-circuits:QFN50P350X350X100-21N-D, symbol SolarCellX_v3-rescue:BQ25570RGRR-misc-circuits-cache-misc-circuits-rescue
- J2: symbol symbols:U.FL-R-SMT-1 -> SolarCell+Y-rescue:U.FL-R-SMT-1-symbols
- U1: symbol symbols:TTB12G51-Balun -> SolarCell+Y-rescue:TTB12G51-Balun-symbols
- U3: symbol symbols:TSL2561 -> SolarCell+Y-rescue:TSL2561-symbols
Connections:
- net labels added: +3V3, VBAT, VBAT_OK, VOUT_EN
- wire segments 77 -> 177
Other:
- note added: "80% MPPT"
- note added: "BQ25570RGRR"
- note added: "DNI"
- note added: "Energy Harvesting IC"
- note added: "External energy storage\nInput/Output"
- note added: "External\nPower Source\nInput\n(Solar)"
- note added: "Imin=280uA"
- note added: "MPPT Set Resistors"
- note added: "Sets of resistor dividers should = 13MOhm"
- note added: "VBAT_OK\nON: 3.51V\nOFF: 3.42V"
- note added: "VBAT_OV\n4.2V"
- note added: "VOUT=1.21V*((ROUT2+ROUT1)/ROUT1)"
- note added: "VOUT\n3.31"
- note added: "ZENER"
- moved on the sheet: C1, D3, H1, H2, J1, J2, JP1, Q1, R1, R10, R2, R3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
