File: SolarCell+Y.kicad_pcb (KiCad board)
At the start: 6 copper layers, 50 x 50 mm, 27 parts, among them IC1 symbols_TSL2561, Q1 IRLML2803

Commit message: Massaged J1 into there somehow.
Parts:
- added J1: symbols_XF2M-1015-1A, solarpcb:XF2M-1015-1A, F.Cu at (164.5, 58.0)
- IC1: footprint custom-footprints:TSL2561 -> solarpcb:TSL2561
Connections:
- IC1 pad 1: (no net) -> +3V3
- IC1 pad 2: (no net) -> Net-(IC1-Pad2)
- IC1 pad 3: (no net) -> GND
- IC1 pad 4: (no net) -> SCL1
- IC1 pad 6: (no net) -> SDA1
- R1 pad 1: (no net) -> +3V3
- R4 pad 1: (no net) -> BATT_N
- R7 pad 2: (no net) -> BATT_P
Routing:
- net (no net): track 83.2 -> 41.1 mm, vias 7 -> 4
- net +3V3: track 2.24 -> 27.0 mm, vias 0 -> 1
- net SDA1: track 0.00 -> 14.9 mm, vias 0 -> 1
- net SCL1: track 0.00 -> 12.4 mm, vias 0 -> 1
- net Net-(H1-Pad1): track 11.2 -> 0.00 mm
- net Net-(IC1-Pad2): track 3.87 -> 5.22 mm

Commit message: Caught mistake on burnwire circuit.
Parts:
- added J2: U.FL-R-SMT-1, Connector_Coaxial:U.FL_Hirose_U.FL-R-SMT-1_Vertical, B.Cu at (185.1, 74.7)
- R5: value 10k -> 1M
- R7: value 100k -> 1M
Connections:
- R5 pad 1: BURN1 -> Net-(Q1-Pad1)

Commit message: Trace correction.
Routing:
- net BURN1: track 2.47 -> 0.00 mm
- net Net-(Q1-Pad1): track 1.80 -> 3.93 mm
Other:
- board text removed: "v00"
Changed lines of the file:
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@@
   (general
     (thickness 1.6)
-    (drawings 22)
+    (drawings 21)
     (tracks 1613)
     (zones 0)
@@
   (gr_line (start 166.8145 71.247) (end 166.497 71.247) (layer F.SilkS) (width 0.12))
   (gr_line (start 168.021 71.247) (end 167.7035 71.247) (layer F.SilkS) (width 0.12))
-  (gr_text v00 (at 307.6575 133.2865) (layer B.Mask)
-    (effects (font (size 1.5 1.5) (thickness 0.3)) (justify mirror))
-  )
   (gr_text 3V3 (at 150.622 61.468 90) (layer F.SilkS)
     (effects (font (size 0.635 0.635) (thickness 0.127)))
@@
   (segment (start 188.535 63.55) (end 188.085 64) (width 0.2286) (layer Bottom) (net 23))
   (segment (start 189.7 63.55) (end 188.535 63.55) (width 0.2286) (layer Bottom) (net 23))
+  (segment (start 188.085 66.03) (end 188.015 66.1) (width 0.2286) (layer Bottom) (net 23))
+  (segment (start 188.085 64) (end 188.085 66.03) (width 0.2286) (layer Bottom) (net 23))
   (segment (start 152.4405 58.877) (end 152.4635 58.854) (width 0.29972) (layer Top) (net 24))
   (segment (start 152.4405 60.198) (end 152.4405 58.877) (width 0.29972) (layer Top) (net 24))
@@
   (segment (start 190.201309 69.216309) (end 192.02369 69.216309) (width 0.2286) (layer Bottom) (net 24))
   (segment (start 189.385 68.4) (end 190.201309 69.216309) (width 0.2286) (layer Bottom) (net 24))
-  (segment (start 187.115 65.2) (end 188.015 66.1) (width 0.2286) (layer Bottom) (net 25))
-  (segment (start 187.115 64) (end 187.115 65.2) (width 0.2286) (layer Bottom) (net 25))
   (segment (start 192.6 75.3) (end 194.8 73.1) (width 0.6096) (layer Bottom) (net 26))
   (segment (start 190 75.3) (end 192.6 75.3) (width 0.6096) (layer Bottom) (net 26))

Commit message: v01 order + repo update
Parts:
- removed the D1 at (194.4, 64.2)
- removed the H2 at (198.1, 69.4)
- removed the H2 at (198.0, 66.8)
- removed the H2 at (198.1, 64.1)
- removed the H2 at (198.0, 60.0)
- removed the H2 at (198.1, 57.2)
- removed the H2 at (198.1, 54.6)
- removed IC1: symbols_TSL2561, solarpcb:TSL2561
- removed the R1 at (192.1, 68.7)
- removed the R2 at (188.9, 68.4)
- removed the R4 at (192.2, 67.2)
- removed the R5 at (188.5, 66.1)
- removed the R6 at (187.6, 64.0)
- removed the R7 at (192.4, 64.2)
- added C1: 1uF, Capacitor_SMD:C_0402_1005Metric, F.Cu at (154.4, 61.6)
- added C1: 0.1uF, Capacitor_SMD:C_0402_1005Metric, B.Cu at (166.0, 53.0)
- added C1: 1.0uF, Capacitor_SMD:C_0402_1005Metric, B.Cu at (170.7, 56.9)
- added C10: 0.1uF, Capacitor_SMD:C_0402_1005Metric, B.Cu at (167.3, 50.6)
- added C11: 100uF, Capacitor_SMD:C_0603_1608Metric, B.Cu at (176.2, 47.6)
- added C12: 100uF, Capacitor_SMD:C_0603_1608Metric, B.Cu at (165.9, 49.3)
- added C13: 0.1uF, Capacitor_SMD:C_0402_1005Metric, B.Cu at (167.3, 53.0)
- added C14: 100uF, Capacitor_SMD:C_0603_1608Metric, B.Cu at (162.9, 52.5)
- added C2: 0.1uF, Capacitor_SMD:C_0402_1005Metric, B.Cu at (183.4, 47.6)
- added C3: 4.7uF, Capacitor_SMD:C_0402_1005Metric, B.Cu at (180.1, 55.0)
- added C4: 10nF, Capacitor_SMD:C_0402_1005Metric, B.Cu at (180.1, 57.5)
- added C6: 100uF, Capacitor_SMD:C_0603_1608Metric, B.Cu at (170.8, 58.9)
- added C7: 22uF, Capacitor_SMD:C_0402_1005Metric, B.Cu at (171.9, 54.1)
- added C8: 4.7uF, Capacitor_SMD:C_0402_1005Metric, B.Cu at (176.2, 51.1)
- added C9: 0.1uF, Capacitor_SMD:C_0402_1005Metric, B.Cu at (176.2, 49.1)
- added D1: SBDiode, SolarCellParts:SB Diode, F.Cu at (194.3, 53.3)
- added D1: SDM20U40-7, misc-circuits:SOD523, B.Cu at (182.8, 54.9)
- added D2: MSS1P4-M3_89A, custom-footprints:MICROSMP, B.Cu at (169.0, 51.4)
- added D3: MSS1P4-M3_89A, custom-footprints:MICROSMP, B.Cu at (183.6, 50.4)
- added JP1: Jumper, custom-footprints:Burn-Wire, F.Cu at (197.9, 62.2)
- added L1: 22uH-LPS4018-223MR, misc-circuits:LPS4018, B.Cu at (180.3, 50.9)
- added L2: 10uH-LPS4018-103MR, misc-circuits:LPS4018, B.Cu at (172.4, 50.9)
- added R1: 0, Resistor_SMD:R_0402_1005Metric, F.Cu at (154.0, 60.5)
- added R1: 0, Resistor_SMD:R_0402_1005Metric, B.Cu at (172.7, 55.9)
- added R10: 8.25M, Resistor_SMD:R_0402_1005Metric, B.Cu at (172.7, 58.2)
- added R11: 4.75M, Resistor_SMD:R_0402_1005Metric, B.Cu at (172.7, 56.9)
- added R14: 0, Resistor_SMD:R_0402_1005Metric, B.Cu at (180.1, 56.3)
- added R15: 0, Resistor_SMD:R_0402_1005Metric, B.Cu at (181.3, 47.6)
- added R16: 0, Resistor_SMD:R_0402_1005Metric, B.Cu at (179.1, 47.6)
- added R17: 0, Resistor_SMD:R_0402_1005Metric, B.Cu at (169.6, 60.2)
- added R19: 0, Resistor_SMD:R_0402_1005Metric, B.Cu at (163.1, 47.7)
- added R2: 0, Resistor_SMD:R_0402_1005Metric, F.Cu at (154.9, 60.5)
- added R2: 0, Resistor_SMD:R_0402_1005Metric, B.Cu at (161.7, 48.7)
- added R4: 0, Resistor_SMD:R_0402_1005Metric, B.Cu at (168.4, 59.7)
- added R4: 0, Resistor_SMD:R_0402_1005Metric, B.Cu at (163.1, 48.7)
- added R5: 1M, Resistor_SMD:R_0402_1005Metric, B.Cu at (190.2, 51.7)
- added R5: 7.32M, Resistor_SMD:R_0402_1005Metric, B.Cu at (177.8, 59.9)
- added R6: 4.7k, Resistor_SMD:R_0402_1005Metric, B.Cu at (189.7, 53.6)
- added R6: 5.62M, Resistor_SMD:R_0402_1005Metric, B.Cu at (179.6, 59.5)
- added R7: 1M, Resistor_SMD:R_0402_1005Metric, B.Cu at (189.7, 55.6)
- added R7: 374K, Resistor_SMD:R_0402_1005Metric, B.Cu at (176.7, 59.9)
- added R8: 8.25M, Resistor_SMD:R_0402_1005Metric, B.Cu at (175.0, 59.5)
- added R9: 4.53M, Resistor_SMD:R_0402_1005Metric, B.Cu at (172.7, 59.5)
- added Ref**: Val**, custom-footprints:ypanel, F.Cu at (152.4, 92.1)
- added TP1: TP, TestPoint:TestPoint_THTPad_D1.0mm_Drill0.5mm, B.Cu at (180.4, 72.3)
- added TP2: TP, TestPoint:TestPoint_THTPad_D1.0mm_Drill0.5mm, B.Cu at (171.6, 72.3)
- added TP3: TP, TestPoint:TestPoint_THTPad_D1.0mm_Drill0.5mm, B.Cu at (177.0, 72.3)
- added TP4: TP, TestPoint:TestPoint_THTPad_D1.0mm_Drill0.5mm, B.Cu at (184.8, 72.3)
- added TP5: TP, TestPoint:TestPoint_THTPad_D1.0mm_Drill0.5mm, B.Cu at (185.8, 59.5)
- added U1: TTB12G51-Balun, custom-footprints:TTB12G51-balun, B.Cu at (192.4, 76.5)
- added U2: NDS8434, custom-footprints:NDS8434, B.Cu at (191.3, 60.7)
- added U2: Value, misc-circuits:QFN50P350X350X100-21N-D, B.Cu at (176.2, 55.8)
- added U3: TSL2561, custom-footprints:TSL2561, F.Cu at (154.4, 57.7)
- J1: footprint solarpcb:XF2M-1015-1A -> custom-footprints:XF2M-1015-1A; moved to B.Cu
- J2: footprint Connector_Coaxial:U.FL_Hirose_U.FL-R-SMT-1_Vertical -> custom-footprints:U.FL-R-SMT-1
- SC1, SC2, SC3, SC4, SC5, SC6, SC7, SC8: footprint SolarCellParts:KXOB25-05X3F -> custom-footprints:KXOB25-05X3F
- moved R3 35.4 mm to (161.7, 47.7), turned to 270 degrees
- moved Q1 8.20 mm to (192.5, 54.6), turned to 270 degrees
- moved D2 4.43 mm to (154.7, 69.0)
- moved J2 3.58 mm to (188.3, 76.2), turned to 270 degrees
- moved J1 2.54 mm to (166.9, 58.9), turned to 90 degrees
- moved SC1 1.51 mm to (188.0, 67.1)
- moved SC3 1.34 mm to (188.0, 62.7)
- moved SC2 0.87 mm to (179.1, 67.1)
- moved SC7 0.69 mm to (161.3, 88.1)
- moved SC4 0.62 mm to (179.1, 62.7)
- moved SC8 0.56 mm to (170.2, 41.7)
- moved SC5 0.56 mm to (170.2, 88.0)
- moved SC6 0.51 mm to (161.3, 41.7)
Connections:
- H1 pad 1: (no net) -> Net-(H1-Pad1)
- J1 pad 10: (no net) -> COIL_P
- J1 pad 9: (no net) -> COIL_N
- R3 pad 1: (no net) -> /coil
- R3 pad 2: (no net) -> COIL_P
Routing:
- net COIL_P: track 17322.4 -> 13.5 mm, vias 6 -> 2
- net /coil: track 0.00 -> 17299.0 mm, vias 0 -> 7
- net GND: track 27.3 -> 86.7 mm, vias 13 -> 15
- net Net-(D2-Pad2): track 52.9 -> 0.00 mm, vias 11 -> 0
- net (no net): track 41.1 -> 0.00 mm, vias 4 -> 0
- net BATT_P: track 1.78 -> 35.5 mm, vias 0 -> 2
- net BURN1: track 0.00 -> 31.3 mm, vias 0 -> 2
- net +3V3: track 27.0 -> 56.8 mm, vias 1 -> 2
- net Net-(D1-Pad2): track 151.6 -> 122.0 mm
- net /VBAT: track 0.00 -> 14.1 mm, vias 0 -> 2
- net Net-(D1-Pad1): track 45.9 -> 57.9 mm, vias 7 -> 2
- net Net-(R14-Pad1): track 0.00 -> 11.8 mm, vias 0 -> 2
- net VOUT_EN: track 0.00 -> 9.77 mm, vias 0 -> 2
- net Net-(R10-Pad2): track 0.00 -> 6.98 mm, vias 0 -> 2
- net Net-(IC1-Pad2): track 5.22 -> 0.00 mm
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- added copper zone on B.Cu, net /VBURN
- added copper zone on B.Cu, net BATT_P
- added copper zone on B.Cu, net GND
Other:
- rule trace_min: 0.127 -> 0.1524
- board text added: "1"
- board text added: "BURN"
- board text added: "Cable Pinout 1.BATT_P 2.BATT_N 3.SDA 4.SCL 5.BURN 6.3V3 7.GND 8.GND 9.COIL_N 10.COIL_P"
- board text added: "VBAT"
- board text added: "VSOLAR"
- board text added: "v00"
- board text added: "v01"
- board text removed: "Coil +"
- board text removed: "Coil -"

Commit message: fixed unmanufacturable trace clearances and resubmitted order
Parts:
- added REF**: Fiducial_0.75mm_Mask1.5mm, Fiducial:Fiducial_0.75mm_Mask1.5mm, B.Cu at (198.8, 41.1)
- added REF**: Fiducial_0.75mm_Mask1.5mm, Fiducial:Fiducial_0.75mm_Mask1.5mm, F.Cu at (198.8, 41.1)
- added REF**: Fiducial_0.75mm_Mask1.5mm, Fiducial:Fiducial_0.75mm_Mask1.5mm, B.Cu at (151.3, 88.8)
- added REF**: Fiducial_0.75mm_Mask1.5mm, Fiducial:Fiducial_0.75mm_Mask1.5mm, F.Cu at (151.3, 88.8)
- added REF**: Fiducial_0.75mm_Mask1.5mm, Fiducial:Fiducial_0.75mm_Mask1.5mm, B.Cu at (198.8, 88.8)
- added REF**: Fiducial_0.75mm_Mask1.5mm, Fiducial:Fiducial_0.75mm_Mask1.5mm, F.Cu at (198.8, 88.8)
Routing:
- net /coil: track 17299.0 -> 15718.3 mm
Other:
- outline, holes or cut-outs redrawn

Commit message: repaired schematic such that it matches pcb. repaired pcb such that design rules are met
Parts:
- removed C13: 0.1uF, Capacitor_SMD:C_0402_1005Metric
- turned C15 to 270 degrees
- turned R10 to 90 degrees
- turned R3 to 90 degrees
- turned R8 to 90 degrees
- turned R9 to 90 degrees
- renumbered C1 to C15, C1 to C2, C2 to C4, D2 to D4, D1 to D5, R19 to R10, R10 to R12, R1 to R13, R16 to R14, R5 to R15, R6 to R16, R7 to R17, R8 to R18, R9 to R19, R15 to R20, R14 to R21, R17 to R25, R2 to R3, R3 to R8, R4 to R9, U2 to U4
Connections:
- C15 pad 1: GND -> +3V3
- C15 pad 2: +3V3 -> GND
- R10 pad 1: /coil -> COIL_N
- R10 pad 2: COIL_N -> /coil
- R3 pad 1: COIL_P -> /coil
- R3 pad 2: /coil -> COIL_P
- R8 pad 1: /coil -> COIL_P
- R8 pad 2: COIL_P -> /coil
- R9 pad 1: COIL_N -> /coil
- R9 pad 2: /coil -> COIL_N
- U3 pad 5: Net-(U3-Pad5) -> (no net)
Routing:
- net GND: track 86.7 -> 89.9 mm
- net COIL_N: track 11.5 -> 13.2 mm
- net /coil: track 15718.3 -> 15719.4 mm
Other:
- net class Default: trace_width 0.2286 -> 0.127; via_dia 0.5842 -> 0.6; via_drill 0.381 -> 0.3
- rule trace_min: 0.1524 -> 0.127
- rule via_min_size: 0.45 -> 0.6

Commit message: moved burnwire circuit and added slot for fishing twine tiedown
Parts:
- moved R5 5.87 mm to (190.4, 57.5), turned to 180 degrees
- moved JP1 5.25 mm to (198.6, 67.4)
- moved R6 5.04 mm to (190.4, 58.6)
- moved Q1 4.26 mm to (193.2, 58.8)
- moved U2 4.26 mm to (192.0, 64.9)
- moved R7 4.08 mm to (190.4, 59.6)
Routing:
- net GND: track 89.9 -> 72.2 mm, vias 15 -> 14
- net BURN1: track 31.3 -> 26.0 mm, vias 2 -> 1
- net BATT_P: track 35.5 -> 37.5 mm
Other:
- outline, holes or cut-outs redrawn
