File: SolarCell+Y.kicad_pcb (KiCad board)
At the start: 6 copper layers, 50 x 50 mm, 73 parts, among them J1 symbols_XF2M-1015-1A, J2 U.FL-R-SMT-1, Q1 IRLML2803, U1 TTB12G51-Balun, U2 NDS8434, U3 TSL2561, U4 Value

Commit message: Updated magnetorquer coils
Routing:
- net /coil: track 15719.4 -> 13368.3 mm

Commit message: design review and generated gerbers
Other:
- rule pad_to_mask_clearance: 0.0508 -> 0.049
- rule solder_mask_min_width: 0.25 -> 0.099
- board text added: "v02"
