File: SolarCell+Y.kicad_pcb (KiCad board)
At the start: 6 copper layers, 50 x 50 mm, 73 parts, among them J1 symbols_XF2M-1015-1A, J2 U.FL-R-SMT-1, Q1 IRLML2803, U1 TTB12G51-Balun, U2 NDS8434, U3 TSL2561, U4 Value

Commit message: fixed version number, regenerated gerbers and 3d model
Other:
- board text removed: "v01"
Changed lines of the file:
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@@
   (page A4)
   (layers
-    (0 Top signal)
+    (0 Top signal hide)
     (1 In1.Cu signal hide)
     (2 In2.Cu signal hide)
@@
     (36 B.SilkS user)
     (37 F.SilkS user hide)
-    (38 B.Mask user hide)
+    (38 B.Mask user)
     (39 F.Mask user hide)
     (40 Dwgs.User user hide)
@@
   )
   (setup
-    (last_trace_width 0.19)
+    (last_trace_width 0.127)
     (user_trace_width 0.127)
     (user_trace_width 0.16)
@@
       (psa4output false)
       (plotreference true)
-      (plotvalue true)
+      (plotvalue false)
       (plotinvisibletext false)
       (padsonsilk false)
@@
   (gr_line (start 179.1716 55.753) (end 179.1716 56.7436) (layer B.SilkS) (width 0.12))
   (gr_line (start 181.0258 55.753) (end 179.1716 55.753) (layer B.SilkS) (width 0.12))
-  (gr_text v01 (at 174.2186 41.7068 180) (layer B.Mask)
+  (gr_text v02 (at 174.2186 41.7068 180) (layer B.Mask)
     (effects (font (size 1.5 1.5) (thickness 0.3)) (justify mirror))
   )
-  (gr_text v01 (at 151.765 78.74 270) (layer F.Mask)
+  (gr_text v02 (at 151.765 78.74 270) (layer F.Mask)
     (effects (font (size 1.5 1.5) (thickness 0.3)))
   )
@@
     (effects (font (size 1.5 1.5) (thickness 0.3)) (justify mirror))
   )
-  (gr_text v01 (at 151.765 78.74 270) (layer Top)
+  (gr_text v02 (at 151.765 78.74 270) (layer Top)
     (effects (font (size 1.5 1.5) (thickness 0.3)))
   )

Commit message: Fixed magnetorquer coils
Routing:
- net /coil: track 13368.3 -> 13222.1 mm
